File: KiCad/neodk_v1.kicad_sch (KiCad schematic)
At the start: 73 parts, among them J1 FTSH-105-XX-X-DV, J2 Power 5V..12V DC, J3 FC68131, J4 S2B-XH-A(LF)(SN), J5 S2B-XH-A(LF)(SN), Q1 IRLML6344TRPBF, Q2 IRLML6344TRPBF, Q3 PMV50EPEAR, SW2 FSMRA6JH, U1 SGM61410XN6G/TR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

Commit message: Add KiCad project. Board not checked!
Connections:
- net BUCK_EN: now also U1.4 (EN)
- net TRIAC_1: now also U3.15 (PB0)
- net TRIAC_2: now also U3.16 (PB1)
- net TRIAC_3: now also U3.17 (PB2)
- net GNDBREAK: no longer names the net of J2.GNDBREAK
- no-connect marks 0 -> 16
Other:
- note removed: "3.3V"
