File: Eagle_CAD/neodk_v1.3.brd (EAGLE design)
At the start: 80 x 41 mm, 73 parts, among them J1 SWD, J2 Power 5V..12V DC, J3 FC68131, J4 S2B-XH-A(LF)(SN), J5 S2B-XH-A(LF)(SN), Q1 IRLML6344TRPBF, Q2 IRLML6344TRPBF, Q3 PMV50EPEAR, SW2 FSMRA6JH, U1 SGM61410XN6G/TR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

Commit message: Production files for hardware v1.3.
Parts:
- R1, R9: value 150 -> 300
- moved TP3 3.37 mm to (49.6, 13.6)
- moved Q3 1.10 mm to (14.0, 14.9), turned to 0 degrees
Connections:
- net N$30: now also Q3.3; no longer Q3.2
- net VBAT: now also Q3.2; no longer Q3.3
Routing:
- net N$31: track 2.00 -> 4.34 mm
- net N$30: track 1.80 -> 3.95 mm
- net VBAT: track 23.0 -> 24.5 mm
- net N$9: track 15.0 -> 13.9 mm
Other:
- board text added: "NeoDK v1.3 © 2024 Neostim"
- board text removed: "NeoDK v1.2 © 2024 Neostim"
