File: Eagle_CAD/neodk_v1.3.sch (EAGLE design)
At the start: 73 parts, among them J1 SWD, J2 Power 5V..12V DC, J3 FC68131, J4 S2B-XH-A(LF)(SN), J5 S2B-XH-A(LF)(SN), Q1 IRLML6344TRPBF, Q2 IRLML6344TRPBF, Q3 PMV50EPEAR, SW2 FSMRA6JH, U1 SGM61410XN6G/TR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

Commit message: Production files for hardware v1.3.
Parts:
- R1, R9: value 150 -> 300
Other:
- note added: "NeoDK v1.3 © 2024 Neostim"
- note removed: "NeoDK v1.2 © 2024 Neostim"
Changed lines of the file:
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@@
 <part name="R7" library="rcl" library_urn="urn:adsk.eagle:library:334" deviceset="R-EU_" device="R0603" package3d_urn="urn:adsk.eagle:package:23555/3" value="300"/>
 <part name="R8" library="rcl" library_urn="urn:adsk.eagle:library:334" deviceset="R-EU_" device="R0603" package3d_urn="urn:adsk.eagle:package:23555/3" value="300"/>
-<part name="R9" library="rcl" library_urn="urn:adsk.eagle:library:334" deviceset="R-EU_" device="R0603" package3d_urn="urn:adsk.eagle:package:23555/3" value="150"/>
-<part name="R1" library="rcl" library_urn="urn:adsk.eagle:library:334" deviceset="R-EU_" device="R0603" package3d_urn="urn:adsk.eagle:package:23555/3" value="150"/>
+<part name="R9" library="rcl" library_urn="urn:adsk.eagle:library:334" deviceset="R-EU_" device="R0603" package3d_urn="urn:adsk.eagle:package:23555/3" value="300"/>
+<part name="R1" library="rcl" library_urn="urn:adsk.eagle:library:334" deviceset="R-EU_" device="R0603" package3d_urn="urn:adsk.eagle:package:23555/3" value="300"/>
 <part name="R2" library="rcl" library_urn="urn:adsk.eagle:library:334" deviceset="R-EU_" device="R0603" package3d_urn="urn:adsk.eagle:package:23555/3" value="300"/>
 <part name="SUPPLY2" library="supply2" library_urn="urn:adsk.eagle:library:372" deviceset="VCC" device=""/>
@@
 <text x="195.58" y="53.34" size="2.286" layer="91" ratio="12">Use ONLY
 this transformer.</text>
-<text x="132.08" y="48.26" size="2.286" layer="91" ratio="10">NeoDK v1.2
+<text x="132.08" y="48.26" size="2.286" layer="91" ratio="10">NeoDK v1.3
 © 2024 Neostim</text>
 <text x="91.44" y="-20.32" size="1.778" layer="91">ADC</text>
